File: Game Console/Game Console.kicad_pcb (KiCad board)
At the start: 2 copper layers, 124.9 x 52.2 mm, 14 parts, among them SW1 SW_UP, SW2 SW_DOWN, SW3 SW_LEFT, SW4 SW_RIGHT, SW5 SW_A, SW6 SW_B

Commit message: Updated all files for the newest version of the project
Parts:
- added FT232RLFTDI1: Conn_01x06_Pin, Connector_PinHeader_2.54mm:PinHeader_1x06_P2.54mm_Vertical, F.Cu at (166.5, 88.1)
- moved Ard-PM1 50.0 mm to (139.5, 108.5)
- moved BZ1 33.5 mm to (91.9, 78.5)
- moved UP 18.3 mm to (98.0, 93.0)
- moved G*** 17.6 mm to (139.9, 87.5)
- moved LEFT 16.8 mm to (88.5, 100.5)
- moved RIGHT 16.1 mm to (107.5, 100.5)
- moved DOWN 14.8 mm to (98.0, 108.0)
- moved SSD1306 9.93 mm to (136.4, 71.0)
- moved B 4.21 mm to (171.5, 110.0)
- moved A 0.70 mm to (183.5, 100.5)
- renumbered SW5 to A, SW6 to B, SW2 to DOWN, SW3 to LEFT, SW4 to RIGHT, SW1 to UP
Connections:
- Ard-PM1 pad DTR: unconnected-(Ard-PM1-PadDTR) -> Net-(FT232RLFTDI1-Pin_6)
- Ard-PM1 pad GND1: Net-(Ard-PM1-GND-PadGND1) -> GND
- Ard-PM1 pad RXI: unconnected-(Ard-PM1-PadRXI) -> Net-(FT232RLFTDI1-Pin_5)
- Ard-PM1 pad TXO: unconnected-(Ard-PM1-PadTXO) -> Net-(FT232RLFTDI1-Pin_4)
Routing:
- net Net-(FT232RLFTDI1-Pin_6): track 0.00 -> 92.1 mm, vias 0 -> 2
- net Net-(FT232RLFTDI1-Pin_5): track 0.00 -> 89.0 mm, vias 0 -> 1
- net VCC: track 35.5 -> 113.8 mm, vias 1 -> 0
- net Net-(FT232RLFTDI1-Pin_4): track 0.00 -> 71.9 mm, vias 0 -> 1
- net Net-(Ard-PM1-4): track 108.4 -> 65.7 mm, vias 1 -> 0
- net Net-(Ard-PM1-3): track 88.2 -> 46.6 mm
- net Net-(Ard-PM1-2): track 92.3 -> 56.1 mm, vias 2 -> 3
- net GND: track 10.3 -> 45.6 mm, vias 1 -> 4
- net Net-(Ard-PM1-5): track 84.5 -> 52.7 mm, vias 1 -> 0
- net Net-(Ard-PM1-6): track 19.1 -> 49.4 mm, vias 1 -> 0
- net Net-(Ard-PM1-9): track 104.4 -> 78.4 mm
- net Net-(SSD1306-Pin_4): track 48.0 -> 34.8 mm, vias 2 -> 0
- net Net-(SSD1306-Pin_3): track 46.6 -> 34.8 mm, vias 1 -> 0
- net Net-(Ard-PM1-7): track 35.7 -> 30.9 mm
