File: Game Console/Game Console.kicad_sch (KiCad schematic)
At the start: 9 parts, among them SW1 SW_UP, SW2 SW_DOWN, SW3 SW_LEFT, SW4 SW_RIGHT, SW5 SW_A, SW6 SW_B

Commit message: Updated all files for the newest version of the project
Parts:
- added FT232RLFTDI1: Conn_01x06_Pin, Connector_PinHeader_2.54mm:PinHeader_1x06_P2.54mm_Vertical, symbol Connector:Conn_01x06_Pin
Connections:
- net GND: now also Ard-PM1.GND1 (GND), FT232RLFTDI1.1 (Pin_1), FT232RLFTDI1.2 (Pin_2)
- net VCC: now also FT232RLFTDI1.3 (Pin_3)
- net at Ard-PM1.DTR: now also FT232RLFTDI1.6 (Pin_6)
- net at Ard-PM1.RXI: now also FT232RLFTDI1.5 (Pin_5)
- net at Ard-PM1.TXO: now also FT232RLFTDI1.4 (Pin_4)
- no-connect marks 4 -> 1
Other:
- moved on the sheet: Ard-PM1, BZ1, SSD1306, SW1, SW2, SW3, SW4, SW5, SW6
